File: ayab-esp32/aux-connectors.kicad_sch (KiCad schematic)
At the start: 27 parts, among them J801 AYAB_UART, J802 I2C_VBUS, J803 USER_I2C, J804 I2C_VBUS, J805 AYAB_SPI, J806 AYAB_I2C, Q801 AO3400A, Q802 AO3400A, Q803 AO3400A, Q804 AO3400A

Commit message: Close Rev A independent audit repair order
Parts:
- added R209, R210: 5k1, Resistor_SMD:R_0603_1608Metric, symbol ayab-lib:R_Small_US
Connections:
- net +3V3: now also R209.1, R210.1
- net AYAB_SCL: now also R209.2
- net AYAB_SDA: now also R210.2
Changed lines of the file:
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@@
+    )
+  )
+  (label "AYAB_SCL" (at 147.32 91.44 0) (fields_autoplaced)
+    (effects (font (size 1.27 1.27)) (justify left bottom))
+  )
+  (label "AYAB_SDA" (at 160.02 91.44 0) (fields_autoplaced)
+    (effects (font (size 1.27 1.27)) (justify left bottom))
+  )
+  (symbol (lib_id "power:+3V3") (at 147.32 86.36 0) (unit 1)
+    (in_bom yes) (on_board yes) (dnp no)
+    (property "Reference" "#PWR0820" (at 147.32 90.17 0)
+      (effects (font (size 1.27 1.27)) hide)
+    )
+    (property "Value" "+3V3" (at 147.32 82.55 0)
+      (effects (font (size 1.27 1.27)))
+    )
+    (property "Footprint" "" (at 147.32 86.36 0)
+      (effects (font (size 1.27 1.27)) hide)
+    )
+    (property "Datasheet" "" (at 147.32 86.36 0)
+      (effects (font (size 1.27 1.27)) hide)
+    )
+    (pin "1")
+    (instances
+      (project "ayab-esp32"
+        (path "/ad16b75f-afc8-4717-a7c6-8dd7b69a18e2/b41a48c7-b009-4c26-92ce-a01689c1d02b"
+          (reference "#PWR0820") (unit 1)
+        )
+      )
+    )
+  )
+  (symbol (lib_id "power:+3V3") (at 160.02 86.36 0) (unit 1)
+    (in_bom yes) (on_board yes) (dnp no)
+    (property "Reference" "#PWR0821" (at 160.02 90.17 0)
+      (effects (font (size 1.27 1.27)) hide)
+    )
+    (property "Value" "+3V3" (at 160.02 82.55 0)
+      (effects (font (size 1.27 1.27)))
+    )
+    (property "Footprint" "" (at 160.02 86.36 0)
+      (effects (font (size 1.27 1.27)) hide)
+    )
+    (property "Datasheet" "" (at 160.02 86.36 0)
+      (effects (font (size 1.27 1.27)) hide)
+    )
+    (pin "1")
+    (instances
+      (project "ayab-esp32"
+        (path "/ad16b75f-afc8-4717-a7c6-8dd7b69a18e2/b41a48c7-b009-4c26-92ce-a01689c1d02b"
+          (reference "#PWR0821") (unit 1)
+        )
+      )
+    )
+  )
+(symbol (lib_id "ayab-lib:R_Small_US") (at 147.32 88.9 0) (unit 1)
+    (in_bom yes) (on_board yes) (dnp no)
+    (property "Reference" "R209" (at 146.05 87.63 0)
+      (effects (font (size 1.27 1.27)) (justify right))
+    )
+    (property "Value" "5k1" (at 146.05 90.17 0)
+      (effects (font (size 1.27 1.27)) (justify right))
+    )
+    (property "Footprint" "Resistor_SMD:R_0603_1608Metric" (at 147.32 88.9 0)
+      (effects (font (size 1.27 1.27)) hide)
+    )
+    (property "Datasheet" "~" (at 147.32 88.9 0)
+      (effects (font (size 1.27 1.27)) hide)
+    )
+    (property "LCSC ID" "C23186" (at 147.32 88.9 0)
+      (effects (font (size 1.27 1.27)) hide)
+    )
+    (property "Voltage rating" "" (at 147.32 88.9 0)
+      (effects (font (size 1.27 1.27)) hide)
+    )
+    (property "Package" "0603" (at 147.32 88.9 0)
+      (effects (font (size 1.27 1.27)) hide)
+    )
+    (property "OEM PN" "0603WAF5101T5E" (at 147.32 88.9 0)
+      (effects (font (size 1.27 1.27)) hide)
+    )
+    (property "OEM" "UNI-ROYAL(Uniroyal Elec)" (at 147.32 88.9 0)
+      (effects (font (size 1.27 1.27)) hide)
+    )
+    (pin "1")
+    (pin "2")
+    (instances
+      (project "ayab-esp32"
+        (path "/ad16b75f-afc8-4717-a7c6-8dd7b69a18e2/b41a48c7-b009-4c26-92ce-a01689c1d02b"
+          (reference "R209") (unit 1)
+        )
+      )
+    )
+  )
+(symbol (lib_id "ayab-lib:R_Small_US") (at 160.02 88.9 0) (unit 1)
+    (in_bom yes) (on_board yes) (dnp no)
+    (property "Reference" "R210" (at 158.75 87.63 0)
+      (effects (font (size 1.27 1.27)) (justify right))
+    )
+    (property "Value" "5k1" (at 158.75 90.17 0)
+      (effects (font (size 1.27 1.27)) (justify right))
+    )
+    (property "Footprint" "Resistor_SMD:R_0603_1608Metric" (at 160.02 88.9 0)
+      (effects (font (size 1.27 1.27)) hide)
+    )
+    (property "Datasheet" "~" (at 160.02 88.9 0)
+      (effects (font (size 1.27 1.27)) hide)
+    )
+    (property "LCSC ID" "C23186" (at 160.02 88.9 0)
+      (effects (font (size 1.27 1.27)) hide)
+    )
+    (property "Voltage rating" "" (at 160.02 88.9 0)
+      (effects (font (size 1.27 1.27)) hide)
+    )
+    (property "Package" "0603" (at 160.02 88.9 0)
+      (effects (font (size 1.27 1.27)) hide)
+    )
+    (property "OEM PN" "0603WAF5101T5E" (at 160.02 88.9 0)
+      (effects (font (size 1.27 1.27)) hide)
+    )
+    (property "OEM" "UNI-ROYAL(Uniroyal Elec)" (at 160.02 88.9 0)
+      (effects (font (size 1.27 1.27)) hide)
+    )
+    (pin "1")
+    (pin "2")
+    (instances
+      (project "ayab-esp32"
+        (path "/ad16b75f-afc8-4717-a7c6-8dd7b69a18e2/b41a48c7-b009-4c26-92ce-a01689c1d02b"
+          (reference "R210") (unit 1)
+        )
+      )
     )
   )
