File: ayab-esp32/ayab-esp32.kicad_pcb (KiCad board)
At the start: 4 copper layers, 285.1 x 48.1 mm, 236 parts, among them J201 SPARE1, J202 SPARE0, J401 900.965.CK35 SOLENOIDS A, J402 900.965.CK35 SOLENOIDS B, J403 910.950 SOLENOIDS A, J404 910.950 SOLENOIDS B, J405 910.950 ENCODERS EOL R, J406 930.940 SOLENOIDS A, J407 930.940 SOLENOIDS B, J408 910.950 EOL L, J409 930.940 EOL R, J410 930.940 ENCODERS, J411 900.965 EOL L, J412 900.965 EOL R, J413 900.965 ENCODERS, J414 930.940 EOL L, J501 USB_C_Receptacle_USB2.0, J601 VIN, J602 Brother_5P, J604 Brother_4R, J701 CTRL_3v3, J702 CTRL_5V, J801 AYAB_UART, J802 I2C_VBUS, J803 USER_I2C, J804 I2C_VBUS, J805 AYAB_SPI, J806 AYAB_I2C, Q201 AO3400A, Q501 BCM857BV, Q502 LP9435LT1G, Q801 AO3400A, Q802 AO3400A, Q803 AO3400A, Q804 AO3400A, Q805 LP9435LT1G, Q806 AO3400A, SW201 USER, SW202 RESET, SW203 BOOTSEL, U201 ESP32-S3-MINI-1, U301 MCP23017_SS, U302 ULN2003A, U303 ULN2003A, U304 ULN2003A, U403 LM66100DCKR, U501 SRV05-4, U601 XL1509, U602 XL1509, U701 SN74LVC4245

Commit message: Integrate protected machine-power sensing
Parts:
- added C206: 100n, Capacitor_SMD:C_0603_1608Metric, B.Cu at (237.2, 160.5)
- added D205: CDBU0130-HF, Diode_SMD:D_0603_1608Metric, B.Cu at (234.0, 157.0)
- added D206: CDBU0130-HF, Diode_SMD:D_0603_1608Metric, B.Cu at (234.0, 160.5)
Routing:
- net /ESP32/MACHINE_PWR_SENSE: track 63.4 -> 78.1 mm
- net +3V3: track 512.2 -> 518.4 mm

Commit message: Close Rev A independent audit repair order
Parts:
- removed kibuzzard-65BDBF94: G***, kibuzzard-65BDBF94
- removed kibuzzard-65BFE062: G***, kibuzzard-65BFE062
- TP701: value CMP-L -> HALL-L-RAW
- TP702: value CMP-R -> HALL-R-RAW
Connections:
- net /ESP32/EOL_L_N renamed Net-(J701-Pin_5)
- net /ESP32/EOL_L_P renamed Net-(J701-Pin_4)
- net /ESP32/EOL_R_N renamed Net-(J701-Pin_7)
- net /ESP32/ESP14 renamed /ESP32/FRONT_PANEL_AUX
- net /ESP32/ESP39 renamed /ESP32/PANEL_INT
- net /IO CONDITIONING/EOL_L_K renamed Net-(J702-Pin_4)
- net /IO CONDITIONING/EOL_L_L renamed Net-(J702-Pin_5)
- net Net-(U201-SPIIO7/GPIO36/FSPICLK/SUBSPICLK) renamed /ESP32/USER_BUTTON
- J701 pad 6: /ESP32/EOL_R_P -> Net-(J701-Pin_6)
- U201 pad 7: /ESP32/EOL_R_P -> unconnected-(U201-GPIO3/TOUCH3/ADC1_CH2-Pad7)
- U403 pad 4: (no net) -> unconnected-(U403-N/C-Pad4)
- U701 pad 16: /ESP32/EOL_R_P -> Net-(J701-Pin_6)
Routing:
- net /ESP32/EOL_R_P: track 78.0 -> 0.00 mm, vias 1 -> 0
- net Net-(J701-Pin_6): track 0.00 -> 18.6 mm
Other:
- board text added: "D205 K=3V3"
- board text added: "D206 A=GND"
- board text added: "KH910 REV A 09/2026"
- board text added: "SOLENOID GATE"
- board text added: "TP703 SW"
