File: ayab-esp32/ioconditioning.kicad_sch (KiCad schematic)
At the start: 25 parts, among them J701 CTRL_3v3, J702 CTRL_5V, U701 SN74LVC4245

Commit message: Integrate protected machine-power sensing
Parts:
- C701, C702: LCSC ID C57112 -> C14663; OEM FH (Guangdong Fenghua Advanced Tech) -> Samsung Electro-Mechanics; OEM PN 0603B103K500NT -> CL10B104KB8NNNC; Voltage rating 24V X7R -> 50V X7R
Changed lines of the file:
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@@
       (effects (font (size 1.27 1.27)) hide)
     )
-    (property "Voltage rating" "24V X7R" (at 66.04 76.2 0)
-      (effects (font (size 1.27 1.27)) hide)
-    )
-    (property "LCSC ID" "C57112" (at 66.04 76.2 0)
-      (effects (font (size 1.27 1.27)) hide)
-    )
-    (property "OEM PN" "0603B103K500NT" (at 66.04 76.2 0)
-      (effects (font (size 1.27 1.27)) hide)
-    )
-    (property "OEM" "FH (Guangdong Fenghua Advanced Tech)" (at 66.04 76.2 0)
+    (property "Voltage rating" "50V X7R" (at 66.04 76.2 0)
+      (effects (font (size 1.27 1.27)) hide)
+    )
+    (property "LCSC ID" "C14663" (at 66.04 76.2 0)
+      (effects (font (size 1.27 1.27)) hide)
+    )
+    (property "OEM PN" "CL10B104KB8NNNC" (at 66.04 76.2 0)
+      (effects (font (size 1.27 1.27)) hide)
+    )
+    (property "OEM" "Samsung Electro-Mechanics" (at 66.04 76.2 0)
       (effects (font (size 1.27 1.27)) hide)
     )
@@
       (effects (font (size 1.27 1.27)) hide)
     )
-    (property "Voltage rating" "24V X7R" (at 157.48 77.47 0)
-      (effects (font (size 1.27 1.27)) hide)
-    )
-    (property "LCSC ID" "C57112" (at 157.48 77.47 0)
-      (effects (font (size 1.27 1.27)) hide)
-    )
-    (property "OEM PN" "0603B103K500NT" (at 157.48 77.47 0)
-      (effects (font (size 1.27 1.27)) hide)
-    )
-    (property "OEM" "FH (Guangdong Fenghua Advanced Tech)" (at 157.48 77.47 0)
-      (effects (font (size 1.27 1.27)) hide)
-    )
+    (property "Voltage rating" "50V X7R" (at 157.48 77.47 0)
+      (effects (font (size 1.27 1.27)) hide)
+    )
+    (property "LCSC ID" "C14663" (at 157.48 77.47 0)
+      (effects (font (size 1.27 1.27)) hide)
+    )
+    (property "OEM PN" "CL10B104KB8NNNC" (at 157.48 77.47 0)
+      (effects (font (size 1.27 1.27)) hide)
+    )
+    (property "OEM" "Samsung Electro-Mechanics" (at 157.48 77.47 0)
+      (effects (font (size 1.27 1.27)) hide)
+    )

Commit message: Close Rev A independent audit repair order
Connections:
- net EOL_L_K: no longer names the net of J702.4 (Pin_4), R707.1, R708.2, U701.6 (A4)
- net EOL_L_L: no longer names the net of J702.5 (Pin_5), R709.1, R710.2, U701.7 (A5)
