File: ayab-esp32/ayab-esp32.kicad_sch (KiCad schematic)
At the start: 14 parts

Commit message: Bypass KH910 K-L comparators and add pull-ups
Other:
- sheet ESP32 ports: added KH910_R_K, KH910_R_L; removed none
- sheet IO CONDITIONING ports: added none; removed EOL_R_K, EOL_R_L
Changed lines of the file:
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@@
   (wire (pts (xy 68.58 46.99) (xy 68.58 49.53))
     (stroke (width 0) (type default))
-  )
-  (wire (pts (xy 200.66 147.32) (xy 219.71 147.32))
-    (stroke (width 0) (type default))
-  )
-  (wire (pts (xy 140.97 44.45) (xy 219.71 44.45))
+  )  (wire (pts (xy 140.97 44.45) (xy 219.71 44.45))
     (stroke (width 0) (type default))
   )
@@
   (wire (pts (xy 76.2 134.62) (xy 76.2 146.05))
     (stroke (width 0) (type default))
-  )
-  (wire (pts (xy 200.66 144.78) (xy 219.71 144.78))
-    (stroke (width 0) (type default))
-  )
-  (wire (pts (xy 60.96 74.93) (xy 97.79 74.93))
+  )  (wire (pts (xy 60.96 74.93) (xy 97.79 74.93))
     (stroke (width 0) (type default))
   )
@@
     )
   )
+  (wire (pts (xy 219.71 144.78) (xy 215.9 144.78))
+    (stroke (width 0) (type default))
+  )
+  (wire (pts (xy 215.9 144.78) (xy 215.9 160.02))
+    (stroke (width 0) (type default))
+  )
+  (wire (pts (xy 215.9 160.02) (xy 146.05 160.02))
+    (stroke (width 0) (type default))
+  )
+  (wire (pts (xy 146.05 160.02) (xy 146.05 149.86))
+    (stroke (width 0) (type default))
+  )
+  (wire (pts (xy 146.05 149.86) (xy 140.97 149.86))
+    (stroke (width 0) (type default))
+  )
+  (wire (pts (xy 219.71 147.32) (xy 218.44 147.32))
+    (stroke (width 0) (type default))
+  )
+  (wire (pts (xy 218.44 147.32) (xy 218.44 162.56))
+    (stroke (width 0) (type default))
+  )
+  (wire (pts (xy 218.44 162.56) (xy 148.59 162.56))
+    (stroke (width 0) (type default))
+  )
+  (wire (pts (xy 148.59 162.56) (xy 148.59 152.4))
+    (stroke (width 0) (type default))
+  )
+  (wire (pts (xy 148.59 152.4) (xy 140.97 152.4))
+    (stroke (width 0) (type default))
+  )
   (sheet (at 34.29 26.67) (size 26.67 27.94) (fields_autoplaced)
     (stroke (width 0.1524) (type solid))
@@
       (effects (font (size 1.27 1.27)) (justify right))
     )
-    (pin "EOL_R_K" input (at 200.66 144.78 0)
-      (effects (font (size 1.27 1.27)) (justify right))
-    )
-    (pin "EOL_R_L" input (at 200.66 147.32 0)
-      (effects (font (size 1.27 1.27)) (justify right))
-    )
-    (pin "EOL_L_N" output (at 160.02 147.32 180)
+            (pin "EOL_L_N" output (at 160.02 147.32 180)
       (effects (font (size 1.27 1.27)) (justify left))
     )
@@
       (effects (font (size 1.27 1.27)) (justify right))
     )
+    (pin "KH910_R_K" input (at 140.97 149.86 0)
+      (effects (font (size 1.27 1.27)) (justify right))
+    )
+    (pin "KH910_R_L" input (at 140.97 152.4 0)
+      (effects (font (size 1.27 1.27)) (justify right))
+    )

Commit message: Add passive analog Hall ADC paths
Other:
- sheet ESP32 ports: added HALL_L_ADC, HALL_R_ADC; removed EOL_L_N, EOL_L_P, EOL_R_N, EOL_R_P
- sheet IO CONDITIONING ports: added HALL_L_ADC, HALL_R_ADC; removed EOL_L_N, EOL_L_P, EOL_R_N, EOL_R_P
Changed lines of the file:
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@@
   (wire (pts (xy 66.04 143.51) (xy 66.04 146.05))
     (stroke (width 0) (type default))
-  )
-  (wire (pts (xy 140.97 139.7) (xy 160.02 139.7))
-    (stroke (width 0) (type default))
-  )
-  (wire (pts (xy 55.88 134.62) (xy 66.04 134.62))
+  )  (wire (pts (xy 55.88 134.62) (xy 66.04 134.62))
     (stroke (width 0) (type default))
   )
@@
   (wire (pts (xy 60.96 86.36) (xy 66.04 86.36))
     (stroke (width 0) (type default))
-  )
-  (wire (pts (xy 140.97 142.24) (xy 160.02 142.24))
-    (stroke (width 0) (type default))
-  )
-  (wire (pts (xy 200.66 124.46) (xy 219.71 124.46))
+  )  (wire (pts (xy 200.66 124.46) (xy 219.71 124.46))
     (stroke (width 0) (type default))
   )
@@
       (effects (font (size 1.27 1.27)) (justify right))
     )
-            (pin "EOL_L_N" output (at 160.02 147.32 180)
-      (effects (font (size 1.27 1.27)) (justify left))
-    )
-    (pin "EOL_R_P" output (at 160.02 139.7 180)
-      (effects (font (size 1.27 1.27)) (justify left))
-    )
-    (pin "EOL_R_N" output (at 160.02 142.24 180)
-      (effects (font (size 1.27 1.27)) (justify left))
-    )
-    (pin "EOL_L_P" output (at 160.02 144.78 180)
+            (pin "HALL_R_ADC" output (at 160.02 147.32 180)
+      (effects (font (size 1.27 1.27)) (justify left))
+    )
+            (pin "HALL_L_ADC" output (at 160.02 144.78 180)
       (effects (font (size 1.27 1.27)) (justify left))
     )
@@
       (effects (font (size 1.27 1.27)) (justify left))
     )
-    (pin "EOL_L_P" input (at 140.97 144.78 0)
+    (pin "HALL_L_ADC" input (at 140.97 144.78 0)
       (effects (font (size 1.27 1.27)) (justify right))
     )
-    (pin "EOL_L_N" input (at 140.97 147.32 0)
+    (pin "HALL_R_ADC" input (at 140.97 147.32 0)
       (effects (font (size 1.27 1.27)) (justify right))
     )
-    (pin "EOL_R_P" input (at 140.97 139.7 0)
+            (pin "I2C0_SDA" bidirectional (at 140.97 93.98 0)
       (effects (font (size 1.27 1.27)) (justify right))
     )
-    (pin "EOL_R_N" input (at 140.97 142.24 0)
-      (effects (font (size 1.27 1.27)) (justify right))
-    )
-    (pin "I2C0_SDA" bidirectional (at 140.97 93.98 0)
-      (effects (font (size 1.27 1.27)) (justify right))
-    )

Commit message: Close final Rev A preorder audit findings
Parts:
- H101, H102, H103, H104, H106, H108: value M3 -> M2
Changed lines of the file:
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@@
       (effects (font (size 1.27 1.27)) (justify left))
     )
-    (property "Value" "M3" (at 48.26 129.54 0)
+    (property "Value" "M2" (at 48.26 129.54 0)
       (effects (font (size 1.27 1.27)) (justify left))
     )
@@
       (effects (font (size 1.27 1.27)) (justify left))
     )
-    (property "Value" "M3" (at 58.42 129.54 0)
+    (property "Value" "M2" (at 58.42 129.54 0)
       (effects (font (size 1.27 1.27)) (justify left))
     )
@@
       (effects (font (size 1.27 1.27)) (justify left))
     )
-    (property "Value" "M3" (at 68.58 140.97 0)
+    (property "Value" "M2" (at 68.58 140.97 0)
       (effects (font (size 1.27 1.27)) (justify left))
     )
@@
       (effects (font (size 1.27 1.27)) (justify left))
     )
-    (property "Value" "M3" (at 68.58 129.54 0)
+    (property "Value" "M2" (at 68.58 129.54 0)
       (effects (font (size 1.27 1.27)) (justify left))
     )
@@
       (effects (font (size 1.27 1.27)) (justify left))
     )
-    (property "Value" "M3" (at 58.42 140.97 0)
+    (property "Value" "M2" (at 58.42 140.97 0)
       (effects (font (size 1.27 1.27)) (justify left))
     )
@@
       (effects (font (size 1.27 1.27)) (justify left))
     )
-    (property "Value" "M3" (at 48.26 140.97 0)
-      (effects (font (size 1.27 1.27)) (justify left))
-    )
+    (property "Value" "M2" (at 48.26 140.97 0)
+      (effects (font (size 1.27 1.27)) (justify left))
+    )
