File: ayab-esp32/mcu.kicad_sch (KiCad schematic)
At the start: 34 parts, among them J201 SPARE1, J202 SPARE0, Q201 AO3400A, SW201 USER, SW202 RESET, SW203 BOOTSEL, U201 ESP32-S3-MINI-1

Commit message: Close Rev A independent audit repair order
Connections:
- net USER_BUTTON: now reaches C201.1, R201.2, SW201.1, U201.32 (SPIIO7/GPIO36/FSPICLK/SUBSPICLK)
- net ESP14 renamed FRONT_PANEL_AUX
- net ESP39 renamed PANEL_INT
Changed lines of the file:
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@@
   (no_connect (at 259.08 44.45))
   (no_connect (at 93.98 115.57))
-  (label "SOLENOID_PWR_EN" (at 195.58 115.57 0) (fields_autoplaced)
-    (effects (font (size 1.27 1.27)) (justify left bottom))
-  )
   (global_label "SOLENOID_PWR_EN" (shape output) (at 203.2 115.57 0) (fields_autoplaced)
     (effects (font (size 1.27 1.27)) (justify left))
@@
     (effects (font (size 1.27 1.27)) (justify left bottom))
   )
-  (wire (pts (xy 205.74 82.55) (xy 220.98 82.55))
+  (label "FRONT_PANEL_AUX" (at 185.42 107.95 0) (fields_autoplaced)
+    (effects (font (size 1.27 1.27)) (justify left bottom))
+  )
+  (label "PANEL_INT" (at 93.98 69.85 180) (fields_autoplaced)
+    (effects (font (size 1.27 1.27)) (justify right bottom))
+  )
+  (label "USER_BUTTON" (at 93.98 125.73 180) (fields_autoplaced)
+    (effects (font (size 1.27 1.27)) (justify right bottom))
+  )
+  (wire (pts (xy 205.74 82.55) (xy 213.36 82.55))
+    (stroke (width 0) (type default))
+  )
+  (wire (pts (xy 213.36 82.55) (xy 220.98 82.55))
     (stroke (width 0) (type default))
   )
@@
     (effects (font (size 1.27 1.27)) (justify left bottom))
   )
-  (label "ESP39" (at 82.5122 69.85 0) (fields_autoplaced)
-    (effects (font (size 1.27 1.27)) (justify left bottom))
-  )
   (label "BOOT1" (at 82.55 184.15 0) (fields_autoplaced)
     (effects (font (size 1.27 1.27)) (justify left bottom))
@@
     (effects (font (size 1.27 1.27)) (justify right bottom))
   )
-  (label "ESP14" (at 198.12 107.95 180) (fields_autoplaced)
-    (effects (font (size 1.27 1.27)) (justify right bottom))
-  )
   (label "BUZZER" (at 232.41 63.5 0) (fields_autoplaced)
     (effects (font (size 1.27 1.27)) (justify left bottom))
   )
-  (label "ESP21" (at 198.12 115.57 180) (fields_autoplaced)
-    (effects (font (size 1.27 1.27)) (justify right bottom))
-  )
   (hierarchical_label "KH910_R_L" (shape input) (at 198.12 113.03 0) (fields_autoplaced)
     (effects (font (size 1.27 1.27)) (justify left))
@@
     (instances
       (project "ayab-esp32"
-        (path "/ad16b75f-afc8-4717-a7c6-8dd7b69a18e2/aaa14c5f-6969-439e-bdef-bb5fc66f917d"
+        (path "/ad16b75f-afc8-4717-a7c6-8dd7b69a18e2/a7e0db0f-e473-44d4-a2fe-681f732aacb2"
           (reference "D205") (unit 1)
         )
@@
     (instances
       (project "ayab-esp32"
-        (path "/ad16b75f-afc8-4717-a7c6-8dd7b69a18e2/175ec455-5c18-4495-952f-cdd672f0311a"
+        (path "/ad16b75f-afc8-4717-a7c6-8dd7b69a18e2/a7e0db0f-e473-44d4-a2fe-681f732aacb2"
           (reference "D206") (unit 1)
         )
@@
     (instances
       (project "ayab-esp32"
-        (path "/ad16b75f-afc8-4717-a7c6-8dd7b69a18e2/86d7191f-1078-449e-8193-ca35bc117e8d"
+        (path "/ad16b75f-afc8-4717-a7c6-8dd7b69a18e2/a7e0db0f-e473-44d4-a2fe-681f732aacb2"
           (reference "C206") (unit 1)
         )

Commit message: Close final Rev A preorder audit findings
Parts:
- D204: OEM (none) -> MDD (Microdiode Semiconductor)
Changed lines of the file:
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@@
       (effects (font (size 1.27 1.27)) hide)
     )
-    (property "Datasheet" "~" (at 247.65 41.91 0)
+    (property "Datasheet" "https://datasheet.lcsc.com/datasheet/pdf/8a09f89034087b5d1623ed150a6cce5b.pdf?productCode=C22452" (at 247.65 41.91 0)
+      (effects (font (size 1.27 1.27)) hide)
+    )
+    (property "Description" "SS54 5 A 40 V SMA Schottky rectifier" (at 247.65 41.91 0)
       (effects (font (size 1.27 1.27)) hide)
     )
@@
       (effects (font (size 1.27 1.27)) hide)
     )
-    (property "OEM" "" (at 247.65 41.91 0)
+    (property "OEM" "MDD (Microdiode Semiconductor)" (at 247.65 41.91 0)
       (effects (font (size 1.27 1.27)) hide)
     )
@@
       (effects (font (size 1.27 1.27)) hide)
     )
+    (property "Description" "CDBU0130-HF 30 V low-leakage Schottky diode" (at 213.36 78.74 0)
+      (effects (font (size 1.27 1.27)) hide)
+    )
     (property "Package" "0603/SOD-523F" (at 213.36 78.74 0)
       (effects (font (size 1.27 1.27)) hide)
@@
       (effects (font (size 1.27 1.27)) hide)
     )
+    (property "Description" "CDBU0130-HF 30 V low-leakage Schottky diode" (at 213.36 86.36 0)
+      (effects (font (size 1.27 1.27)) hide)
+    )
