File: ayab-esp32/solenoids.kicad_sch (KiCad schematic)
At the start: 17 parts, among them Q805 LP9435LT1G, Q806 AO3400A, U301 MCP23017_SS

Commit message: Integrate protected machine-power sensing
Parts:
- C301, C305: LCSC ID C57112 -> C14663; OEM FH (Guangdong Fenghua Advanced Tech) -> Samsung Electro-Mechanics; OEM PN 0603B103K500NT -> CL10B104KB8NNNC; Voltage rating 24V X7R -> 50V X7R
Changed lines of the file:
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@@
       (effects (font (size 1.27 1.27)) hide)
     )
-    (property "Voltage rating" "24V X7R" (at 69.85 54.61 0)
-      (effects (font (size 1.27 1.27)) hide)
-    )
-    (property "LCSC ID" "C57112" (at 69.85 54.61 0)
-      (effects (font (size 1.27 1.27)) hide)
-    )
-    (property "OEM PN" "0603B103K500NT" (at 69.85 54.61 0)
-      (effects (font (size 1.27 1.27)) hide)
-    )
-    (property "OEM" "FH (Guangdong Fenghua Advanced Tech)" (at 69.85 54.61 0)
+    (property "Voltage rating" "50V X7R" (at 69.85 54.61 0)
+      (effects (font (size 1.27 1.27)) hide)
+    )
+    (property "LCSC ID" "C14663" (at 69.85 54.61 0)
+      (effects (font (size 1.27 1.27)) hide)
+    )
+    (property "OEM PN" "CL10B104KB8NNNC" (at 69.85 54.61 0)
+      (effects (font (size 1.27 1.27)) hide)
+    )
+    (property "OEM" "Samsung Electro-Mechanics" (at 69.85 54.61 0)
       (effects (font (size 1.27 1.27)) hide)
     )
@@
       (effects (font (size 1.27 1.27)) hide)
     )
-    (property "Voltage rating" "24V X7R" (at 59.69 54.61 0)
-      (effects (font (size 1.27 1.27)) hide)
-    )
-    (property "LCSC ID" "C57112" (at 59.69 54.61 0)
-      (effects (font (size 1.27 1.27)) hide)
-    )
-    (property "OEM PN" "0603B103K500NT" (at 59.69 54.61 0)
-      (effects (font (size 1.27 1.27)) hide)
-    )
-    (property "OEM" "FH (Guangdong Fenghua Advanced Tech)" (at 59.69 54.61 0)
-      (effects (font (size 1.27 1.27)) hide)
-    )
+    (property "Voltage rating" "50V X7R" (at 59.69 54.61 0)
+      (effects (font (size 1.27 1.27)) hide)
+    )
+    (property "LCSC ID" "C14663" (at 59.69 54.61 0)
+      (effects (font (size 1.27 1.27)) hide)
+    )
+    (property "OEM PN" "CL10B104KB8NNNC" (at 59.69 54.61 0)
+      (effects (font (size 1.27 1.27)) hide)
+    )
+    (property "OEM" "Samsung Electro-Mechanics" (at 59.69 54.61 0)
+      (effects (font (size 1.27 1.27)) hide)
+    )

Commit message: Close Rev A independent audit repair order
Changed lines of the file:
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@@
     (effects (font (size 1.27 1.27)) (justify left))
-  )
-  (label "SOLENOID_12V_SW" (at 243.84 167.64 0) (fields_autoplaced)
-    (effects (font (size 1.27 1.27)) (justify left bottom))
   )
   (junction (at 228.6 167.64) (diameter 0) (color 0 0 0 0)

Commit message: Close final Rev A preorder audit findings
Parts:
- gave numbers to parts that had none: 3
