File: ayab-esp32/brother-connectors.kicad_sch (KiCad schematic)
At the start: 16 parts, among them J401 900.965.CK35 SOLENOIDS A, J402 900.965.CK35 SOLENOIDS B, J403 910.950 SOLENOIDS A, J404 910.950 SOLENOIDS B, J405 910.950 ENCODERS EOL R, J406 930.940 SOLENOIDS A, J407 930.940 SOLENOIDS B, J408 910.950 EOL L, J409 930.940 EOL R, J410 930.940 ENCODERS, J411 900.965 EOL L, J412 900.965 EOL R, J413 900.965 ENCODERS, J414 930.940 EOL L

Commit message: Add hardware-default-OFF solenoid power gate
Connections:
- net +12V renamed SOLENOID_12V_SW
Changed lines of the file:
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@@
     (stroke (width 0) (type default))
+  )
+  (global_label "SOLENOID_12V_SW" (shape input) (at 55.88 34.29 0) (fields_autoplaced)
+    (effects (font (size 1.27 1.27)) (justify left))
+  )
+  (global_label "SOLENOID_12V_SW" (shape input) (at 144.78 34.29 0) (fields_autoplaced)
+    (effects (font (size 1.27 1.27)) (justify left))
+  )
+  (global_label "SOLENOID_12V_SW" (shape input) (at 234.95 36.83 0) (fields_autoplaced)
+    (effects (font (size 1.27 1.27)) (justify left))
   )
   (wire (pts (xy 133.35 128.27) (xy 147.32 128.27))
@@
         (path "/ad16b75f-afc8-4717-a7c6-8dd7b69a18e2/7cdcbcc1-4c9b-4f2f-a9ba-c3dab0b4149d"
           (reference "J404") (unit 1)
-        )
-      )
-    )
-  )
-  (symbol (lib_id "power:+12V") (at 144.78 34.29 0) (unit 1)
-    (in_bom yes) (on_board yes) (dnp no) (fields_autoplaced)
-    (property "Reference" "#PWR0404" (at 144.78 38.1 0)
-      (effects (font (size 1.27 1.27)) hide)
-    )
-    (property "Value" "+12V" (at 144.78 29.21 0)
-      (effects (font (size 1.27 1.27)))
-    )
-    (property "Footprint" "" (at 144.78 34.29 0)
-      (effects (font (size 1.27 1.27)) hide)
-    )
-    (property "Datasheet" "" (at 144.78 34.29 0)
-      (effects (font (size 1.27 1.27)) hide)
-    )
-    (pin "1")
-    (instances
-      (project "ayab-esp32"
-        (path "/ad16b75f-afc8-4717-a7c6-8dd7b69a18e2/7cdcbcc1-4c9b-4f2f-a9ba-c3dab0b4149d"
-          (reference "#PWR0404") (unit 1)
         )
       )
@@
     )
   )
-  (symbol (lib_id "power:+12V") (at 234.95 36.83 0) (unit 1)
-    (in_bom yes) (on_board yes) (dnp no) (fields_autoplaced)
-    (property "Reference" "#PWR0406" (at 234.95 40.64 0)
-      (effects (font (size 1.27 1.27)) hide)
-    )
-    (property "Value" "+12V" (at 234.95 31.75 0)
-      (effects (font (size 1.27 1.27)))
-    )
-    (property "Footprint" "" (at 234.95 36.83 0)
-      (effects (font (size 1.27 1.27)) hide)
-    )
-    (property "Datasheet" "" (at 234.95 36.83 0)
-      (effects (font (size 1.27 1.27)) hide)
-    )
-    (pin "1")
-    (instances
-      (project "ayab-esp32"
-        (path "/ad16b75f-afc8-4717-a7c6-8dd7b69a18e2/7cdcbcc1-4c9b-4f2f-a9ba-c3dab0b4149d"
-          (reference "#PWR0406") (unit 1)
-        )
-      )
-    )
-  )
   (symbol (lib_id "ayab-lib:Conn_01x10") (at 152.4 49.53 0) (mirror x) (unit 1)
     (in_bom yes) (on_board yes) (dnp no)
@@
         )
       )
-    )
-  )
-  (symbol (lib_id "power:+12V") (at 55.88 34.29 0) (unit 1)
-    (in_bom yes) (on_board yes) (dnp no) (fields_autoplaced)
-    (property "Reference" "#PWR0401" (at 55.88 38.1 0)
-      (effects (font (size 1.27 1.27)) hide)
-    )
-    (property "Value" "+12V" (at 55.88 29.21 0)
-      (effects (font (size 1.27 1.27)))
-    )
-    (property "Footprint" "" (at 55.88 34.29 0)
-      (effects (font (size 1.27 1.27)) hide)
-    )
-    (property "Datasheet" "" (at 55.88 34.29 0)
-      (effects (font (size 1.27 1.27)) hide)
-    )
-    (pin "1")
-    (instances
-      (project "ayab-esp32"
-        (path "/ad16b75f-afc8-4717-a7c6-8dd7b69a18e2/7cdcbcc1-4c9b-4f2f-a9ba-c3dab0b4149d"
-          (reference "#PWR0401") (unit 1)
-        )
-      )

Commit message: Approve available tin J404 and document display interface
Parts:
- J404: OEM PN HNC2-2.5P-8DS(02) -> HNC2-2.5P-8DS(55)
Changed lines of the file:
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@@
       (effects (font (size 1.27 1.27)) hide)
     )
-    (property "OEM PN" "HNC2-2.5P-8DS(02)" (at 152.4 77.47 0)
+    (property "OEM PN" "HNC2-2.5P-8DS(55)" (at 152.4 77.47 0)
       (effects (font (size 1.27 1.27)) hide)
     )
